File: pcb/v0.2/microscope.kicad_pcb (KiCad board)
At the start: 2 copper layers, 19 x 100.2 mm, 0 parts

Commit message: changes lol
Parts:
- added C1: 10n, Capacitor_SMD:C_0805_2012Metric, F.Cu at (123.8, 84.8)
- added C2: 470n, Capacitor_SMD:C_0805_2012Metric, F.Cu at (123.8, 87.8)
- added C3: 100n, Capacitor_SMD:C_0805_2012Metric, F.Cu at (123.8, 90.9)
- added C4: 10u, Capacitor_SMD:C_0805_2012Metric, F.Cu at (123.8, 93.9)
- added C5: 100n, Capacitor_SMD:C_0805_2012Metric, F.Cu at (123.8, 96.9)
- added C6: 100n, Capacitor_SMD:C_0805_2012Metric, F.Cu at (123.8, 99.9)
- added C7: 22u, Capacitor_SMD:C_0805_2012Metric, F.Cu at (123.8, 102.9)
- added D1: LED, LED_SMD:LED_PLCC_2835, F.Cu at (114.9, 111.8)
- added D2: MB10S, MB10S:SOIC245P670X290-4N, F.Cu at (135.7, 94.4)
- added D3: D, Diode_SMD:D_SOD-323, F.Cu at (128.2, 113.3)
- added IC1: AL8860QMP-13, KiCad:SOP65P490X110-9N, F.Cu at (115.8, 107.3)
- added J1: Conn_01x02_Socket, Connector_JST:JST_XH_B2B-XH-A_1x02_P2.50mm_Vertical, F.Cu at (115.6, 86.7)
- added J3: Conn_01x03_Socket, Connector_JST:JST_XH_B3B-XH-A_1x03_P2.50mm_Vertical, F.Cu at (129.5, 86.7)
- added L1: L, Inductor_SMD:L_1210_3225Metric, F.Cu at (133.3, 112.6)
- added R1: 1.2, Resistor_SMD:R_0805_2012Metric, F.Cu at (128.3, 92.6)
- added R3: 1k, Resistor_SMD:R_0805_2012Metric, F.Cu at (128.3, 95.6)
- added R4: 51k, Resistor_SMD:R_0805_2012Metric, F.Cu at (128.3, 98.5)
- added R5: 10k, Resistor_SMD:R_0805_2012Metric, F.Cu at (128.3, 101.5)
- added R6: 20k, Resistor_SMD:R_0805_2012Metric, F.Cu at (128.3, 104.4)
- added R7: 20k, Resistor_SMD:R_0805_2012Metric, F.Cu at (128.3, 107.4)
- added R9: 51k, Resistor_SMD:R_0805_2012Metric, F.Cu at (128.3, 110.3)
- added U1: OP07CDR, OP07CDR:SOIC127P599X175-8N, F.Cu at (134.7, 107.3)
- added U2: NE555DR, NE555DR:SOIC127P599X175-8N, F.Cu at (135.2, 100.9)
- added U3: L78L05_SOT89, Package_TO_SOT_SMD:SOT-89-3, F.Cu at (115.5, 102.0)
- added U4: Solder Pad, custom_components:SolderPad_3x3mm, F.Cu at (119.5, 112.0)

Commit message: first commit
Parts:
- added U5: Solder Pad, custom_components:SolderPad_3x3mm, F.Cu at (140.4, 98.6)
- moved D1 64.6 mm to (150.0, 57.5)
- moved U3 47.3 mm to (145.2, 138.8)
- moved J1 43.0 mm to (150.5, 111.8), turned to -90 degrees
- moved U1 40.9 mm to (153.8, 143.5)
- moved J3 40.2 mm to (150.5, 121.0), turned to -90 degrees
- moved IC1 38.3 mm to (152.2, 95.2)
- moved U2 38.2 mm to (153.8, 134.2)
- moved L1 30.3 mm to (152.5, 89.2)
- moved U4 27.0 mm to (140.4, 95.0), turned to 90 degrees
- moved D2 19.1 mm to (152.5, 103.5)
Connections:
- U4 pad 1: unconnected-(U4-Pad1) -> Net-(D1-A)
Other:
- board size 19 x 100.2 mm -> 19 x 96 mm

Commit message: v0.2 pcb finished
Parts:
- removed D1: LED, LED_SMD:LED_PLCC_2835
- removed D3: D, Diode_SMD:D_SOD-323
- removed IC1: AL8860QMP-13, KiCad:SOP65P490X110-9N
- removed L1: L, Inductor_SMD:L_1210_3225Metric
- added C8: 22u, Capacitor_SMD:C_0805_2012Metric, F.Cu at (96.6, 84.8)
- added D4: LED, LED_SMD:LED_PLCC_2835, F.Cu at (100.0, 54.0)
- added D5: D, Diode_SMD:D_SOD-323, F.Cu at (96.0, 81.7)
- added IC2: AL8860QMP-13, KiCad:SOP65P490X110-9N, F.Cu at (101.7, 83.8)
- added L2: 47u, Inductor_SMD:L_1210_3225Metric, F.Cu at (99.9, 79.9)
- added Q1: NPN, custom_components:custom_SOT-23-3, F.Cu at (98.0, 133.2)
- added Q2: PNP, custom_components:custom_SOT-23-3, F.Cu at (98.0, 129.5)
- added R2: 1.2, Resistor_SMD:R_0603_1608Metric, F.Cu at (101.7, 86.7)
- added U10: Solder Pad, custom_components:SolderPad_3x3mm, F.Cu at (109.0, 103.8)
- added U6: LM358DR, LM358DR:SOIC127P599X175-8N, F.Cu at (103.5, 126.1)
- added U7: Solder Pad, custom_components:SolderPad_3x3mm, F.Cu at (109.0, 97.8)
- added U8: Solder Pad, custom_components:SolderPad_3x3mm, F.Cu at (109.0, 95.2)
- added U9: Solder Pad, custom_components:SolderPad_3x3mm, F.Cu at (109.0, 91.8)
- C1, C2, C3, C5, C6: footprint Capacitor_SMD:C_0805_2012Metric -> Capacitor_SMD:C_0603_1608Metric
- C4: value 10u -> 220u; footprint Capacitor_SMD:C_0805_2012Metric -> Capacitor_THT:CP_Radial_D6.3mm_P2.50mm; moved to B.Cu
- C7: value 22u -> 220u; footprint Capacitor_SMD:C_0805_2012Metric -> Capacitor_THT:CP_Radial_D6.3mm_P2.50mm; moved to B.Cu
- R1: value 1.2 -> 1k; footprint Resistor_SMD:R_0805_2012Metric -> Resistor_SMD:R_0603_1608Metric
- R3, R5, R6, R7: footprint Resistor_SMD:R_0805_2012Metric -> Resistor_SMD:R_0603_1608Metric
- R4, R9: value 51k -> 22k; footprint Resistor_SMD:R_0805_2012Metric -> Resistor_SMD:R_0603_1608Metric
- U1: value OP07CDR -> Solder Pad; footprint OP07CDR:SOIC127P599X175-8N -> custom_components:SolderPad_3x3mm
- moved U1 61.5 mm to (109.0, 101.2), turned to -90 degrees
- moved C1 58.5 mm to (95.2, 135.9)
- moved D2 57.4 mm to (96.1, 114.2), turned to 90 degrees
- moved J1 53.1 mm to (100.0, 95.5), turned to 90 degrees
- moved U2 52.9 mm to (101.0, 138.4), turned to 180 degrees
- moved J3 52.6 mm to (100.0, 106.5), turned to 90 degrees
- moved C5 52.0 mm to (98.8, 142.4), turned to 180 degrees
- moved C3 51.9 mm to (106.0, 139.6), turned to -90 degrees
- moved R6 48.0 mm to (95.2, 139.2)
- moved R3 47.9 mm to (94.5, 129.5)
- moved R1 47.5 mm to (101.5, 131.9), turned to 90 degrees
- moved U3 46.9 mm to (105.2, 114.2)
- moved R5 44.9 mm to (94.5, 131.0), turned to 180 degrees
- moved R7 44.8 mm to (95.2, 137.6)
- moved C4 37.1 mm to (97.0, 119.5)
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Connections:
- C3 pad 1: Net-(U1-IN-) -> Net-(U2-THRES)
- R1 pad 1: Net-(D1-A) -> Net-(Q1-B)
- R1 pad 2: VCC -> Net-(U6-1OUT)
- R3 pad 2: Net-(U1-OUT) -> Net-(Q1-E)
- R7 pad 2: Net-(U1-IN-) -> Net-(U2-THRES)
- U1 pad 1: unconnected-(U1-OFFSET_N1-Pad1) -> PWM
- U2 pad 2: Net-(U1-IN-) -> Net-(U2-THRES)
- U2 pad 4: VCC -> +5V
- U2 pad 6: Net-(U1-IN-) -> Net-(U2-THRES)
- U4 pad 1: Net-(D1-A) -> GND
- U5 pad 1: VCC -> Net-(D4-A)
Routing:
- net +5V: track 0.00 -> 74.8 mm, vias 0 -> 4
- net VCC: track 0.00 -> 73.4 mm, vias 0 -> 2
- net Net-(U2-THRES): track 0.00 -> 69.0 mm, vias 0 -> 3
- net PWM: track 0.00 -> 61.0 mm, vias 0 -> 3
- net Net-(J3-Pin_2): track 0.00 -> 56.4 mm, vias 0 -> 2
- net Net-(D4-A): track 0.00 -> 43.8 mm
- net Net-(Q1-B): track 0.00 -> 37.4 mm, vias 0 -> 2
- net Net-(J1-Pin_2): track 0.00 -> 28.6 mm
- net Net-(D4-K): track 0.00 -> 26.1 mm
- net Net-(J1-Pin_1): track 0.00 -> 19.1 mm
- net GND: track 0.00 -> 17.1 mm, vias 0 -> 2
- net Net-(D5-A): track 0.00 -> 8.54 mm
- net Net-(Q1-E): track 0.00 -> 5.29 mm
- net Net-(U2-DISCH): track 0.00 -> 4.84 mm
- net Net-(J3-Pin_3): track 0.00 -> 3.90 mm
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- added copper zone on B.Cu, net GND
- added copper zone on F.Cu, net GND
Other:
- board size 19 x 96 mm -> 19 x 101 mm
- board text added: "GND"
- board text added: "PWM"
- board text added: "R(LED)"
- board text added: "Vin"
- board text added: "Vref"
- board text added: "raw"
