File: PCB/v0.3/microscope.kicad_pcb (KiCad board)
At the start: 2 copper layers, 17 x 90.5 mm, 31 parts, among them IC2 AL8860QMP-13, J1 Conn_01x03_Socket, J3 Conn_01x02_Socket, U2 NE555DR, U3 L78L05_SOT89, U6 LM358DR

Commit message: tweaking
Parts:
- removed C8: 22u, Capacitor_SMD:C_0805_2012Metric
- removed D5: D, Diode_SMD:D_SOD-323
- removed IC2: AL8860QMP-13, KiCad:SOP65P490X110-9N
- removed L2: 47u, Inductor_SMD:L_1210_3225Metric
- removed TP1, TP2: TestPoint_Probe, TestPoint:TestPoint_THTPad_1.0x1.0mm_Drill0.5mm
- removed U3: L78L05_SOT89, Package_TO_SOT_SMD:SOT-89-3
- added Q2: AO3400A, Package_TO_SOT_SMD:SOT-23, F.Cu at (100.2, 74.1)
- added R1: 100, Resistor_SMD:R_0805_2012Metric, F.Cu at (101.8, 70.2)
- added U1: HT75xx-1-SOT89, Package_TO_SOT_SMD:SOT-89-3, F.Cu at (104.4, 113.4)
- C2: value 470n -> 10u
- C6: value 100n -> 10u
- D4: footprint LED_SMD:LED_PLCC_2835 -> led:LED_2835
- GND1: renamed from TP4; footprint TestPoint:TestPoint_THTPad_2.0x2.0mm_Drill1.0mm -> TestPoint:TestPoint_Plated_Hole_D2.0mm
- J1: footprint Connector_JST:JST_XH_S3B-XH-A-1_1x03_P2.50mm_Horizontal -> xh-custom:JST_XH_S3B-A-no-support
- J3: footprint Connector_JST:JST_XH_S2B-XH-A-1_1x02_P2.50mm_Horizontal -> xh-custom:JST_XH_S2B-A-no-support
- PWM1: renamed from TP3; footprint TestPoint:TestPoint_THTPad_2.0x2.0mm_Drill1.0mm -> TestPoint:TestPoint_Plated_Hole_D2.0mm
- R2: value 2.5 -> 100; footprint Resistor_SMD:R_0603_1608Metric -> Resistor_SMD:R_0805_2012Metric
- TP5, TP6: footprint TestPoint:TestPoint_THTPad_2.0x2.0mm_Drill1.0mm -> TestPoint:TestPoint_Plated_Hole_D2.0mm
- moved TP6 43.7 mm to (94.4, 135.1)
- moved TP5 42.2 mm to (94.4, 129.5)
- moved R3 7.40 mm to (104.5, 130.0), turned to -90 degrees
- moved C6 7.20 mm to (104.4, 110.2), turned to 180 degrees
- moved R5 6.41 mm to (102.0, 128.6), turned to 0 degrees
- moved R9 2.93 mm to (101.6, 78.7)
- moved R4 2.92 mm to (101.6, 85.4)
- moved GND1 2.86 mm to (105.7, 87.8)
- moved U6 2.79 mm to (100.9, 133.4), turned to -90 degrees
- moved C2 2.38 mm to (103.6, 117.2)
- moved R2 2.35 mm to (99.5, 70.2)
- moved PWM1 1.30 mm to (105.7, 81.3)
- moved J1 0.56 mm to (99.5, 79.5)
- moved J3 0.54 mm to (99.5, 90.5)
- moved D4 0.42 mm to (100.0, 53.0)
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Connections:
- D4 pad 2: Net-(D4-A) -> +5V
- R2 pad 1: VCC -> Net-(D4-K)
- R2 pad 2: Net-(D4-A) -> Net-(Q2-D)
- TP5 pad 1: Net-(D4-A) -> Net-(J1-Pin_2)
- TP6 pad 1: VCC -> Net-(U2-THRES)
Routing:
- net +5V: track 0.00 -> 92.2 mm
- net PWM: track 0.00 -> 58.4 mm, vias 0 -> 1
- net Net-(J1-Pin_2): track 0.00 -> 58.1 mm, vias 0 -> 1
- net Net-(U2-THRES): track 0.00 -> 30.2 mm, vias 0 -> 3
- net Net-(D4-K): track 0.00 -> 18.9 mm
- net Net-(J3-Pin_1): track 0.00 -> 13.6 mm
- net Net-(J3-Pin_2): track 0.00 -> 9.30 mm
- net Net-(Q2-D): track 0.00 -> 4.43 mm
- net Net-(U2-DISCH): track 0.00 -> 3.79 mm
- net Net-(U2-CONT): track 0.00 -> 2.46 mm
- net Net-(J1-Pin_1): track 0.00 -> 2.27 mm
- net Net-(J1-Pin_3): track 0.00 -> 2.22 mm
- net VCC: track 0.00 -> 1.95 mm
- net Net-(U6-1OUT): track 0.00 -> 1.66 mm
- net GND: vias 0 -> 9
- added copper zone on F.Cu, net +5V
- added copper zone on F.Cu, net PWM
- added copper zone on F.Cu, net VCC
Other:
- board text removed: "GND"
- board text removed: "PWM"
- board text removed: "R(LED)"
- board text removed: "Vpot"
- board text removed: "Vwav"
