File: PCB/v0.3/microscope.kicad_sch (KiCad schematic)
At the start: 31 parts, among them IC2 AL8860QMP-13, J1 Conn_01x03_Socket, J3 Conn_01x02_Socket, U2 NE555DR, U3 L78L05_SOT89, U6 LM358DR

Commit message: tweaking
Parts:
- removed C8: 22u, Capacitor_SMD:C_0805_2012Metric, symbol Device:C
- removed D5: D, Diode_SMD:D_SOD-323, symbol Device:D
- removed IC2: AL8860QMP-13, KiCad:SOP65P490X110-9N, symbol AL8860QMP-13:AL8860QMP-13
- removed L2: 47u, Inductor_SMD:L_1210_3225Metric, symbol Device:L
- removed TP1, TP2: TestPoint_Probe, TestPoint:TestPoint_THTPad_1.0x1.0mm_Drill0.5mm, symbol Connector:TestPoint_Probe
- removed U3: L78L05_SOT89, Package_TO_SOT_SMD:SOT-89-3, symbol Regulator_Linear:L78L05_SOT89
- added Q2: AO3400A, Package_TO_SOT_SMD:SOT-23, symbol Transistor_FET:AO3400A
- added R1: 100, Resistor_SMD:R_0805_2012Metric, symbol Device:R
- added U1: HT75xx-1-SOT89, Package_TO_SOT_SMD:SOT-89-3, symbol Regulator_Linear:HT75xx-1-SOT89
- C2: value 470n -> 10u
- C4, C7: LCSC (none) -> C178534; now in the parts list
- C6: value 100n -> 10u
- D4: footprint LED_SMD:LED_PLCC_2835 -> led:LED_2835; LCSC (none) -> C210319; now in the parts list
- GND1: renamed from TP4; footprint TestPoint:TestPoint_THTPad_2.0x2.0mm_Drill1.0mm -> TestPoint:TestPoint_Plated_Hole_D2.0mm; now left out of the parts list
- J1: footprint Connector_JST:JST_XH_S3B-XH-A-1_1x03_P2.50mm_Horizontal -> xh-custom:JST_XH_S3B-A-no-support; now left out of the parts list
- J3: footprint Connector_JST:JST_XH_S2B-XH-A-1_1x02_P2.50mm_Horizontal -> xh-custom:JST_XH_S2B-A-no-support; now left out of the parts list
- PWM1: renamed from TP3; footprint TestPoint:TestPoint_THTPad_2.0x2.0mm_Drill1.0mm -> TestPoint:TestPoint_Plated_Hole_D2.0mm; now left out of the parts list
- R2: value 2.5 -> 100; footprint Resistor_SMD:R_0603_1608Metric -> Resistor_SMD:R_0805_2012Metric; LCSC (none) -> C17408; now in the parts list
- TP5, TP6: footprint TestPoint:TestPoint_THTPad_2.0x2.0mm_Drill1.0mm -> TestPoint:TestPoint_Plated_Hole_D2.0mm; now left out of the parts list
Connections:
- net +5V: now also D4.2 (A), U1.3 (VOUT)
- net GND: now also Q2.2 (S), U1.1 (GND)
- net PWM: now also Q2.1 (G)
- net VCC: now also U1.2 (VIN); no longer R2.1, TP6.1
- net at J1.2 (Pin_2), U6.3 (1IN+): now also TP5.1
- net at C3.1, R7.2, U2.2 (TRIG)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: now also TP6.1
- net at D4.1 (K): now also R2.1, R1.1
- new net: Q2.3 (D), R1.2, R2.2
Other:
- moved on the sheet: C2, C6, GND1, PWM1
